File: panel_pass-thru/panel_pass-thru.sch (KiCad schematic (older format))
At the start: 2 parts, among them P1 CONN_8, P2 CONN_8

Commit message: improve pass through documentation
Parts:
- P1, P2: symbol pass_thru_panel:CONN_8 -> panel_pass-thru:CONN_8
Changed lines of the file:
@@
 	2050 1850 2950 1850
 $Comp
-L pass_thru_panel:CONN_8 P1
+L panel_pass-thru:CONN_8 P1
 U 1 1 512E7147
 P 1700 1600
@@
 $EndComp
 $Comp
-L pass_thru_panel:CONN_8 P2
+L panel_pass-thru:CONN_8 P2
 U 1 1 512E7142
 P 3300 1600
